Commit message: added new configs for new payload

File: launch/include/config/robot_new.urdf.xacro (robot description, xacro)
@@ -9,9 +9,10 @@
     <origin xyz="0 0 0" rpy="0 0 0" />
   </joint>
-  <link name="xsens_imu"> </link>
+  <link name="vectornav"> </link>
   <joint name="imu_joint" type="fixed">
     <parent link="chassis_link" />
-    <child link="xsens_imu" />
+    <child link="vectornav" />
     <origin xyz="0 0 0" rpy="0 0 0" />
+    <!--origin xyz="0 0 0" rpy="${PI} 0 0" /-->
   </joint>
   <link name="velodyne"> </link>
@@ -20,4 +21,5 @@
     <child link="velodyne" />
     <origin xyz="0 0 0" rpy="0 0 0" />
+    <!--origin xyz="0 0 0" rpy="${PI} 0 0" /-->
   </joint>
   <link name="gps_link"> </link>

Commit message: Working configs

File: launch/include/config/robot_new.urdf.xacro (robot description, xacro)
@@ -27,5 +27,5 @@
     <parent link="chassis_link" />
     <child link="gps_link" />
-    <origin xyz="0 0 0" rpy="0 0 0" />
+    <origin xyz="0 0 0" rpy="${PI} 0 0" />
   </joint>
 </robot>
